File: schematics/si4463-breakout.kicad_pcb (KiCad board)
At the start: 2 copper layers, 23.8 x 34.6 mm, 30 parts, among them J1 HEADER, J2 Coax, U1 Si4463, U2 MAX604, Y1 LFTCXO068373

Commit message: Fix library references
Parts:
- J1: footprint Strix:Breadboard_Header_01x08 -> Strix:Header_Breadboard_1x08
