File: schematics/si4463-breakout.kicad_sch (KiCad schematic)
At the start: 30 parts, among them J1 HEADER, J2 Coax, U1 Si4463, U2 MAX604, Y1 LFTCXO068373

Commit message: Fix library references
Parts:
- J1: footprint Strix:Breadboard_Header_01x08 -> Strix:Header_Breadboard_1x08
Changed lines of the file:
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@@
     (property "Reference" "J1" (id 0) (at 35.56 48.26 0))
     (property "Value" "HEADER" (id 1) (at 35.56 50.8 0))
-    (property "Footprint" "Strix:Breadboard_Header_01x08" (id 2) (at 35.56 62.23 0)
+    (property "Footprint" "Strix:Header_Breadboard_1x08" (id 2) (at 35.56 62.23 0)
       (effects (font (size 1.27 1.27)) hide)
     )
@@
     )
     (path "/41e337e2-8bb5-4b7b-bff1-965426e30326"
-      (reference "J1") (unit 1) (value "HEADER") (footprint "Strix:Breadboard_Header_01x08")
+      (reference "J1") (unit 1) (value "HEADER") (footprint "Strix:Header_Breadboard_1x08")
     )
     (path "/e3f12138-6632-405e-aba7-aaa8ec08b644"
